Commit message: fix urdf generator

File: src/model_generator/robot_data/output/output.urdf (robot description, URDF)
Before this commit: robot raise_a2_t2d0, 3 links, 2 joints
Links:
- added link right_hip_roll, mass 2.39059365; visual mesh filename=file:///home/lizhen/works/open_source/robot_model_generator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 scale=-1.0 1.0 1.0
- added link right_hip_yaw, mass 3.79911511; visual mesh filename=file:///home/lizhen/works/open_source/robot_model_generator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 scale=1.0 -1.0 1.0
- link base_link: geometry visual mesh filename=file:///home/lizhen/works/open_source/robot_model_generator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 scale=1 1 1
- link left_hip_roll: geometry visual mesh filename=file:///home/lizhen/works/open_source/robot_model_generator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 scale=1 1 1
- link left_hip_yaw: geometry visual mesh filename=file:///home/lizhen/works/open_source/robot_model_generator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 scale=1 1 1
Joints:
- added joint idx03_right_hip_roll: type revolute, parent base_link, child right_hip_roll, origin xyz=-0.0808 -0.105 -0.0652 rpy=0.7854 0 1.5708, axis 0 0 1, limit lower=-0.698 upper=0.698 effort=120 velocity=12
- added joint idx04_right_hip_yaw: type revolute, parent right_hip_roll, child right_hip_yaw, origin xyz=-0.0 -0.017 -0.0682 rpy=1.5708 -1.5708 0, axis 0 0 1, limit lower=-1.57 upper=1.57 effort=120 velocity=12

Commit message: add xml generator

File: src/model_generator/robot_data/output/output.urdf (robot description, URDF)
Before this commit: robot raise_a2_t2d0, 5 links, 4 joints
Links:
- link base_link: geometry collision mesh filename=file:///home/lizhen/works/open_source/robot_model_generator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 scale=1 1 1; visual mesh filename=file:///home/lizhen/works/open_source/robot_model_generator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 scale=1 1 1
- link left_hip_roll: geometry collision mesh filename= scale=1 1 1; visual mesh filename=file:///home/lizhen/works/open_source/robot_model_generator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 scale=1 1 1
- link left_hip_yaw: geometry collision mesh filename= scale=1 1 1; visual mesh filename=file:///home/lizhen/works/open_source/robot_model_generator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 scale=1 1 1
- link right_hip_roll: geometry collision mesh filename= scale=-1.0 1.0 1.0; visual mesh filename=file:///home/lizhen/works/open_source/robot_model_generator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 scale=-1.0 1.0 1.0
- link right_hip_yaw: geometry collision mesh filename= scale=1.0 -1.0 1.0; visual mesh filename=file:///home/lizhen/works/open_source/robot_model_generator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 scale=1.0 -1.0 1.0
Joints:
- joint idx01_left_hip_roll: type revolute -> prismatic
- joint idx03_right_hip_roll: type revolute -> prismatic

Commit message: fix bugs

File: src/model_generator/robot_data/output/output.urdf (robot description, URDF)
Before this commit: robot raise_a2_t2d0, 5 links, 4 joints
Links:
- link right_hip_roll: geometry collision mesh filename= scale=1 1 1; visual mesh filename=file:///home/lizhen/works/open_source/robot_model_generator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 scale=-1.0 1.0 1.0
- link right_hip_yaw: geometry collision mesh filename= scale=1 1 1; visual mesh filename=file:///home/lizhen/works/open_source/robot_model_generator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 scale=1.0 -1.0 1.0
Joints:
- joint idx01_left_hip_roll: type prismatic -> revolute
- joint idx03_right_hip_roll: type prismatic -> revolute

Commit message: update

File: src/model_generator/robot_data/output/output.urdf (robot description, URDF)
Before this commit: robot raise_a2_t2d0, 5 links, 4 joints
Links:
- link right_hip_roll: geometry collision mesh filename= scale=1 1 1; visual mesh filename=file:///home/lizhen/works/open_source/robot_model_generator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 scale=1.0 -1.0 1.0
Joints:
- joint idx03_right_hip_roll: origin xyz=-0.0808 -0.105 -0.0652 rpy=0.7854 0 1.5708 -> xyz=-0.0808 -0.105 -0.0652 rpy=-0.7854 0.0 -1.5708
- joint idx04_right_hip_yaw: origin xyz=-0.0 -0.017 -0.0682 rpy=1.5708 -1.5708 0 -> xyz=0.0 0.017 -0.0682 rpy=-1.5708 -1.5708 -0.0

Commit message: update

File: src/model_generator/robot_data/output/output.urdf (robot description, URDF)
Before this commit: robot raise_a2_t2d0, 5 links, 4 joints
Links:
- added link left_arm_link01, mass 0.23884197; collision mesh filename= scale=1 1 1; visual mesh filename=file:///home/lizhen/works/open_source/robot_model_generator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 scale=1 1 1
- added link left_arm_link02, mass 3.09638867; collision mesh filename= scale=1 1 1; visual mesh filename=file:///home/lizhen/works/open_source/robot_model_generator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 scale=1 1 1
- added link left_arm_link03, mass 1.37452988; collision mesh filename= scale=1 1 1; visual mesh filename=file:///home/lizhen/works/open_source/robot_model_generator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 scale=1 1 1
- added link left_arm_link04, mass 0.70457441; collision mesh filename= scale=1 1 1; visual mesh filename=file:///home/lizhen/works/open_source/robot_model_generator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 scale=1 1 1
- added link left_arm_link05, mass 0.12244729; collision mesh filename= scale=1 1 1; visual mesh filename=file:///home/lizhen/works/open_source/robot_model_generator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 scale=1 1 1
- added link left_arm_link06, mass 0.02504627; collision mesh filename= scale=1 1 1; visual mesh filename=file:///home/lizhen/works/open_source/robot_model_generator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 scale=1 1 1
- added link left_arm_link07, mass 0.05050219; collision mesh filename= scale=1 1 1; visual mesh filename=file:///home/lizhen/works/open_source/robot_model_generator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 scale=1 1 1
- added link left_hip_pitch, mass 5.30562514; collision mesh filename= scale=1 1 1; visual mesh filename=file:///home/lizhen/works/open_source/robot_model_generator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 scale=1 1 1
- added link left_knee, mass 2.78469232; collision mesh filename= scale=1 1 1; visual mesh filename=file:///home/lizhen/works/open_source/robot_model_generator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 scale=1 1 1
- added link left_toe_A, mass 0.06362578; collision mesh filename= scale=1 1 1; visual mesh filename=file:///home/lizhen/works/open_source/robot_model_generator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 scale=1 1 1
- added link left_toe_A_rod, mass 0.08203113; collision mesh filename= scale=1 1 1; visual mesh filename=file:///home/lizhen/works/open_source/robot_model_generator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 scale=1 1 1
- added link left_toe_B, mass 0.06362578; collision mesh filename= scale=1 1 1; visual mesh filename=file:///home/lizhen/works/open_source/robot_model_generator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 scale=1 1 1
- added link left_toe_B_rod, mass 0.08225550; collision mesh filename= scale=1 1 1; visual mesh filename=file:///home/lizhen/works/open_source/robot_model_generator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 scale=1 1 1
- added link left_toe_pitch, mass 0.08772028; collision mesh filename= scale=1 1 1; visual mesh filename=file:///home/lizhen/works/open_source/robot_model_generator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 scale=1 1 1
- added link left_toe_roll, mass 0.90432039; collision mesh filename= scale=1 1 1; visual mesh filename=file:///home/lizhen/works/open_source/robot_model_generator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 scale=1 1 1
- added link left_wrist_motor_A, mass 0.22783320; collision mesh filename= scale=1 1 1; visual mesh filename=file:///home/lizhen/works/open_source/robot_model_generator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 scale=1 1 1
- added link left_wrist_motor_B, mass 0.22783320; collision mesh filename= scale=1 1 1; visual mesh filename=file:///home/lizhen/works/open_source/robot_model_generator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 scale=1 1 1
- added link left_wrist_rod_A, mass 0.01468271; collision mesh filename= scale=1 1 1; visual mesh filename=file:///home/lizhen/works/open_source/robot_model_generator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 scale=1 1 1
- added link left_wrist_rod_B, mass 0.01468271; collision mesh filename= scale=1 1 1; visual mesh filename=file:///home/lizhen/works/open_source/robot_model_generator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 scale=1 1 1
- added link right_arm_link01, mass 0.23884197; collision mesh filename= scale=1 1 1; visual mesh filename=file:///home/lizhen/works/open_source/robot_model_generator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 scale=1.0 -1.0 1.0
- added link right_arm_link02, mass 3.09638867; collision mesh filename= scale=1 1 1; visual mesh filename=file:///home/lizhen/works/open_source/robot_model_generator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 scale=1.0 -1.0 1.0
- added link right_arm_link03, mass 1.37452988; collision mesh filename= scale=1 1 1; visual mesh filename=file:///home/lizhen/works/open_source/robot_model_generator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 scale=1.0 -1.0 1.0
- added link right_arm_link04, mass 0.70457441; collision mesh filename= scale=1 1 1; visual mesh filename=file:///home/lizhen/works/open_source/robot_model_generator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 scale=1.0 -1.0 1.0
- added link right_arm_link05, mass 0.12244729; collision mesh filename= scale=1 1 1; visual mesh filename=file:///home/lizhen/works/open_source/robot_model_generator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 scale=1.0 -1.0 1.0
- added link right_arm_link06, mass 0.02504627; collision mesh filename= scale=1 1 1; visual mesh filename=file:///home/lizhen/works/open_source/robot_model_generator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 scale=1.0 -1.0 1.0
- added link right_arm_link07, mass 0.05050219; collision mesh filename= scale=1 1 1; visual mesh filename=file:///home/lizhen/works/open_source/robot_model_generator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 scale=1.0 -1.0 1.0
- added link right_hip_pitch, mass 5.30562514; collision mesh filename= scale=1 1 1; visual mesh filename=file:///home/lizhen/works/open_source/robot_model_generator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 scale=1.0 -1.0 1.0
- added link right_knee, mass 2.78469232; collision mesh filename= scale=1 1 1; visual mesh filename=file:///home/lizhen/works/open_source/robot_model_generator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 scale=1.0 -1.0 1.0
- added link right_toe_A, mass 0.06362578; collision mesh filename= scale=1 1 1; visual mesh filename=file:///home/lizhen/works/open_source/robot_model_generator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 scale=1.0 -1.0 1.0
- added link right_toe_A_rod, mass 0.08203113; collision mesh filename= scale=1 1 1; visual mesh filename=file:///home/lizhen/works/open_source/robot_model_generator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 scale=1.0 -1.0 1.0
- added link right_toe_B, mass 0.06362578; collision mesh filename= scale=1 1 1; visual mesh filename=file:///home/lizhen/works/open_source/robot_model_generator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 scale=1.0 -1.0 1.0
- added link right_toe_B_rod, mass 0.08225550; collision mesh filename= scale=1 1 1; visual mesh filename=file:///home/lizhen/works/open_source/robot_model_generator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 scale=1.0 -1.0 1.0
- added link right_toe_pitch, mass 0.08772028; collision mesh filename= scale=1 1 1; visual mesh filename=file:///home/lizhen/works/open_source/robot_model_generator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 scale=1.0 -1.0 1.0
- added link right_toe_roll, mass 0.90432039; collision mesh filename= scale=1 1 1; visual mesh filename=file:///home/lizhen/works/open_source/robot_model_generator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 scale=1.0 -1.0 1.0
- added link right_wrist_motor_A, mass 0.22783320; collision mesh filename= scale=1 1 1; visual mesh filename=file:///home/lizhen/works/open_source/robot_model_generator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 scale=1.0 -1.0 1.0
- added link right_wrist_motor_B, mass 0.22783320; collision mesh filename= scale=1 1 1; visual mesh filename=file:///home/lizhen/works/open_source/robot_model_generator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 scale=1.0 -1.0 1.0
- added link right_wrist_rod_A, mass 0.01468271; collision mesh filename= scale=1 1 1; visual mesh filename=file:///home/lizhen/works/open_source/robot_model_generator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 scale=1.0 -1.0 1.0
- added link right_wrist_rod_B, mass 0.01468271; collision mesh filename= scale=1 1 1; visual mesh filename=file:///home/lizhen/works/open_source/robot_model_generator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 scale=1.0 -1.0 1.0
Joints:
- removed joint idx03_right_hip_roll
- removed joint idx04_right_hip_yaw
- added joint idx03_left_hip_pitch: type revolute, parent left_hip_yaw, child left_hip_pitch, origin xyz=0 -0.020 0.1205 rpy=1.5708 0.7854 0, axis 0 0 1, limit lower=-1.919862144 upper=0.78539815 effort=140 velocity=12
- added joint idx04_left_knee: type revolute, parent left_hip_pitch, child left_knee, origin xyz=-0.34 0 0 rpy=0 0 0, axis 0 0 1, limit lower=-0.087266461 upper=2.443460911 effort=140 velocity=12
- added joint idx05_left_toe_pitch: type revolute, parent left_knee, child left_toe_pitch, origin xyz=-0.377 0 0 rpy=0 0 0, axis 0 0 1, limit lower=-1.047197533 upper=0.523598767 effort=50 velocity=12
- added joint idx06_left_toe_roll: type revolute, parent left_toe_pitch, child left_toe_roll, origin xyz=0 0 0 rpy=-1.5707963 0 0, axis 0 0 1, limit lower=-0.488692182 upper=0.488692182 effort=50 velocity=12
- added joint idx07_left_toe_A: type fixed, parent left_knee, child left_toe_A, origin xyz=-0.138 0 -0.0315 rpy=0 0 0, axis 0 0 1, limit lower=-1.5708 upper=1.5708 effort=0 velocity=0
- added joint idx08_left_toe_A_rod: type fixed, parent left_toe_A, child left_toe_A_rod, origin xyz=0 -0.063 0 rpy=0 0 0, axis 0 0 1, limit lower=0 upper=0 effort=0 velocity=0
- added joint idx09_left_toe_B: type fixed, parent left_knee, child left_toe_B, origin xyz=-0.232 0 0.0315 rpy=0 0 0, axis 0 0 1, limit lower=-1.5708 upper=1.5708 effort=0 velocity=0
- added joint idx10_left_toe_B_rod: type fixed, parent left_toe_B, child left_toe_B_rod, origin xyz=0 -0.063 0 rpy=0 0 0, axis 0 0 1, limit lower=0 upper=0 effort=0 velocity=0
- added joint idx11_right_hip_roll: type revolute, parent base_link, child right_hip_roll, origin xyz=-0.0808 -0.105 -0.0652 rpy=-0.7854 0.0 -1.5708, axis 0 0 1, limit lower=-0.698 upper=0.698 effort=120 velocity=12
- added joint idx12_right_hip_yaw: type revolute, parent right_hip_roll, child right_hip_yaw, origin xyz=0.0 0.017 -0.0682 rpy=-1.5708 -1.5708 -0.0, axis 0 0 1, limit lower=-1.57 upper=1.57 effort=120 velocity=12
- added joint idx13_right_hip_pitch: type revolute, parent right_hip_yaw, child right_hip_pitch, origin xyz=0.0 0.02 0.1205 rpy=-1.5708 0.7854 -0.0, axis 0 0 1, limit lower=-0.78539815 upper=1.919862144 effort=140 velocity=12
- added joint idx14_right_knee: type revolute, parent right_hip_pitch, child right_knee, origin xyz=-0.34 -0.0 0.0 rpy=-0.0 0.0 -0.0, axis 0 0 1, limit lower=-2.443460911 upper=0.087266461 effort=140 velocity=12
- added joint idx15_right_toe_pitch: type revolute, parent right_knee, child right_toe_pitch, origin xyz=-0.377 -0.0 0.0 rpy=-0.0 0.0 -0.0, axis 0 0 1, limit lower=-0.523598767 upper=1.047197533 effort=50 velocity=12
- added joint idx16_right_toe_roll: type revolute, parent right_toe_pitch, child right_toe_roll, origin xyz=0.0 -0.0 0.0 rpy=1.5707963 0.0 -0.0, axis 0 0 1, limit lower=-0.488692182 upper=0.488692182 effort=50 velocity=12
- added joint idx17_right_toe_A: type fixed, parent right_knee, child right_toe_A, origin xyz=-0.138 -0.0 -0.0315 rpy=-0.0 0.0 -0.0, axis 0 0 1, limit lower=-1.5708 upper=1.5708 effort=0 velocity=0
- added joint idx18_right_toe_A_rod: type fixed, parent right_toe_A, child right_toe_A_rod, origin xyz=0.0 0.063 0.0 rpy=-0.0 0.0 -0.0, axis 0 0 1, limit lower=0 upper=0 effort=0 velocity=0
- added joint idx19_right_toe_B: type fixed, parent right_knee, child right_toe_B, origin xyz=-0.232 -0.0 0.0315 rpy=-0.0 0.0 -0.0, axis 0 0 1, limit lower=-1.5708 upper=1.5708 effort=0 velocity=0
- added joint idx20_right_toe_B_rod: type fixed, parent right_toe_B, child right_toe_B_rod, origin xyz=0.0 0.063 0.0 rpy=-0.0 0.0 -0.0, axis 0 0 1, limit lower=-0.0 upper=-0.0 effort=0 velocity=0
- added joint idx21_left_arm_link01: type revolute, parent base_link, child left_arm_link01, origin xyz=-0.03779 0.191 0.3421 rpy=1.5708 1.5708 0, axis 0 0 1, limit lower=-2.967 upper=2.967 effort=120 velocity=12
- added joint idx22_left_arm_link02: type revolute, parent left_arm_link01, child left_arm_link02, origin xyz=0 0 0 rpy=1.5708 0 0, axis 0 0 1, limit lower=-0.523598767 upper=1.658062761 effort=120 velocity=12
- added joint idx23_left_arm_link03: type revolute, parent left_arm_link02, child left_arm_link03, origin xyz=0 -0.154 0 rpy=1.5708 0 0, axis 0 0 1, limit lower=-2.967 upper=2.967 effort=120 velocity=12
- added joint idx24_left_arm_link04: type revolute, parent left_arm_link03, child left_arm_link04, origin xyz=0 0 0.093 rpy=-1.5708 0 1.5708, axis 0 0 1, limit lower=-2.094395067 upper=0 effort=120 velocity=12
- added joint idx25_left_arm_link05: type revolute, parent left_arm_link04, child left_arm_link05, origin xyz=0 -0.103 0 rpy=1.5708 0 0, axis 0 0 1, limit lower=-2.87979 upper=2.87979 effort=120 velocity=12
- added joint idx26_left_arm_link06: type revolute, parent left_arm_link05, child left_arm_link06, origin xyz=-0.01 0 0.1595 rpy=-1.5708 1.5708 0, axis 0 0 1, limit lower=-0.785398 upper=0.785398 effort=120 velocity=12
- added joint idx27_left_arm_link07: type revolute, parent left_arm_link06, child left_arm_link07, origin xyz=0 0 0 rpy=1.5708 0 0, axis 0 0 1, limit lower=-0.5236 upper=0.5236 effort=120 velocity=12
- added joint idx28_left_wrist_motor_A: type fixed, parent left_arm_link05, child left_wrist_motor_A, origin xyz=0.005 0.02245 0.0245 rpy=0 -3.126778944 0, axis 0 0 1, limit lower=-1.5708 upper=1.5708 effort=120 velocity=12
- added joint idx29_left_wrist_rod_A: type fixed, parent left_wrist_motor_A, child left_wrist_rod_A, origin xyz=0 0.00055 -0.135 rpy=0 3.1415926 0, axis 0 0 1, limit lower=-0.01199 upper=0.01204 effort=120 velocity=12
- added joint idx30_left_wrist_motor_B: type fixed, parent left_arm_link05, child left_wrist_motor_B, origin xyz=0.005 -0.02245 0.0245 rpy=0 -3.126778944 0, axis 0 0 1, limit lower=-1.5708 upper=1.5708 effort=120 velocity=12
- added joint idx31_left_wrist_rod_B: type fixed, parent left_wrist_motor_B, child left_wrist_rod_B, origin xyz=0 0.00055 -0.135 rpy=0 3.1415926 0, axis 0 0 1, limit lower=-0.01199 upper=0.01204 effort=120 velocity=12
- added joint idx32_right_arm_link01: type revolute, parent base_link, child right_arm_link01, origin xyz=-0.03779 -0.191 0.3421 rpy=-1.5708 1.5708 -0.0, axis 0 0 1, limit lower=-2.967 upper=2.967 effort=120 velocity=12
- added joint idx33_right_arm_link02: type revolute, parent right_arm_link01, child right_arm_link02, origin xyz=0.0 -0.0 0.0 rpy=-1.5708 0.0 -0.0, axis 0 0 1, limit lower=-1.658062761 upper=0.523598767 effort=120 velocity=12
- added joint idx34_right_arm_link03: type revolute, parent right_arm_link02, child right_arm_link03, origin xyz=0.0 0.154 0.0 rpy=-1.5708 0.0 -0.0, axis 0 0 1, limit lower=-2.967 upper=2.967 effort=120 velocity=12
- added joint idx35_right_arm_link04: type revolute, parent right_arm_link03, child right_arm_link04, origin xyz=0.0 -0.0 0.093 rpy=1.5708 0.0 -1.5708, axis 0 0 1, limit lower=-0.0 upper=2.094395067 effort=120 velocity=12
- added joint idx36_right_arm_link05: type revolute, parent right_arm_link04, child right_arm_link05, origin xyz=0.0 0.103 0.0 rpy=-1.5708 0.0 -0.0, axis 0 0 1, limit lower=-2.87979 upper=2.87979 effort=120 velocity=12
- added joint idx37_right_arm_link06: type revolute, parent right_arm_link05, child right_arm_link06, origin xyz=-0.01 -0.0 0.1595 rpy=1.5708 1.5708 -0.0, axis 0 0 1, limit lower=-0.785398 upper=0.785398 effort=120 velocity=12
- added joint idx38_right_arm_link07: type revolute, parent right_arm_link06, child right_arm_link07, origin xyz=0.0 -0.0 0.0 rpy=-1.5708 0.0 -0.0, axis 0 0 1, limit lower=-0.5236 upper=0.5236 effort=120 velocity=12
- added joint idx39_right_wrist_motor_A: type fixed, parent right_arm_link05, child right_wrist_motor_A, origin xyz=0.005 -0.02245 0.0245 rpy=-0.0 -3.126778944 -0.0, axis 0 0 1, limit lower=-1.5708 upper=1.5708 effort=120 velocity=12
- added joint idx40_right_wrist_rod_A: type fixed, parent right_wrist_motor_A, child right_wrist_rod_A, origin xyz=0.0 -0.00055 -0.135 rpy=-0.0 3.1415926 -0.0, axis 0 0 1, limit lower=-0.01204 upper=0.01199 effort=120 velocity=12
- added joint idx41_right_wrist_motor_B: type fixed, parent right_arm_link05, child right_wrist_motor_B, origin xyz=0.005 0.02245 0.0245 rpy=-0.0 -3.126778944 -0.0, axis 0 0 1, limit lower=-1.5708 upper=1.5708 effort=120 velocity=12
- added joint idx42_right_wrist_rod_B: type fixed, parent right_wrist_motor_B, child right_wrist_rod_B, origin xyz=0.0 -0.00055 -0.135 rpy=-0.0 3.1415926 -0.0, axis 0 0 1, limit lower=-0.01204 upper=0.01199 effort=120 velocity=12
